Commit message: Customized the Spot Micro robot.
To make it look like the one I made.

File: description/description/urdf/model_spot_micro.urdf.xacro (robot description, xacro)
@@ -1,6 +1,6 @@
 <?xml version="1.0"?>
 <robot xmlns:xacro="http://www.ros.org/wiki/xacro" name="spot_micro">
-  <material name="yellow">
-    <color rgba="0.92 0.83 0.0 1"/>
+  <material name="white">
+    <color rgba="1.0 1.0 1.0 1"/>
   </material>
   <material name="black">
@@ -84,5 +84,5 @@
         <origin rpy="0 -0.139 3.14159" xyz="0.130 0.15 -0.025"/>
         </xacro:unless>
-        <material name="yellow"/>
+        <material name="white"/>
       </visual>
     </link>
@@ -106,5 +106,5 @@
         </geometry>
         <origin rpy="0.0 0.0 0.0" xyz="0.0 0.0 -0.050"/>
-        <material name="yellow"/>-->
+        <material name="white"/>-->
       </visual>
       <collision>
@@ -264,5 +264,5 @@
       </geometry>
       <origin rpy="0 0 3.14159" xyz="0.04 0.055 -0.010"/>
-      <material name="yellow"/>
+      <material name="white"/>
     </visual>
     <collision>
@@ -287,5 +287,5 @@
       </geometry>
       <origin rpy="0 0 3.14159" xyz="0.040 0.055 -0.010"/>
-      <material name="yellow"/>
+      <material name="white"/>
     </visual>
     <collision>

Commit message: Declared the maintainer email & modifed the Spot Micro URDF.
I separated the materials from the robot file, so that I can maybe use them on other future URDF files.

File: description/description/urdf/model_spot_micro.urdf.xacro (robot description, xacro)
@@ -1,13 +1,5 @@
 <?xml version="1.0"?>
 <robot xmlns:xacro="http://www.ros.org/wiki/xacro" name="spot_micro">
-  <material name="white">
-    <color rgba="1.0 1.0 1.0 1"/>
-  </material>
-  <material name="black">
-    <color rgba="0.1 0.1 0.1 1"/>
-  </material>
-  <material name="grey">
-    <color rgba="0.6 0.6 0.6 1"/>
-  </material>
+  <xacro:include filename="materials.xacro"/>
   <!-- Params -->
   <xacro:property name="body_length" value="0.140" />
